File: PCB/omnibot_board/board_v1.sch (EAGLE design)
At the start: 15 parts, among them J1 292303-1

Commit message: New version for OMNI board
Parts:
- J4, J6, J7: SPICEPREFIX (none) -> E
Other:
- note added: "Camera control Arduino Nano"
- note added: "GPIO Digial and analog"
- note added: "I2C connectors"
- note added: "LMI"
- note added: "Motor driver"
- note added: "OMNI BOARD"
- note added: "Power supply"
- moved on the sheet: 12VSOURCE, 5VSOURCE, DRIVER, J1, J10, J2, J3, J4, J5, J6, J7, J8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
