File: PCB/omnibot_board/v1/board_v1.brd (EAGLE design)
At the start: 88.9 x 87.6 mm, 15 parts, among them J1 292303-1

Commit message: changed v1 board
Parts:
- removed J5: (no value), SparkFun-Connectors:1X06
- added J11: (no value), SparkFun-Connectors:1X05
- moved STEPPER 10.9 mm to (41.9, -69.8)
- moved DRIVER 6.35 mm to (41.9, -53.3)
Connections:
- removed net MS1: DRIVER.MS1, NANO.J2.5
- removed net MS2: DRIVER.MS2, NANO.J2.6
- removed net MS3: DRIVER.MS3, NANO.J2.7
- new net A5: J11.3, NANO.J2.7
- new net A6: J11.4, NANO.J2.6
- new net A7: J11.5, NANO.J2.5
- net 3V3: no longer J5.3
- net 5VOLTS: now also J11.2; no longer J5.2
- net A0: now also DRIVER.MS3; no longer J5.4
- net A1: now also DRIVER.MS2; no longer J5.5
- net A2: now also DRIVER.MS1; no longer J5.6
- net GND: now also J11.1; no longer J5.1
Routing:
- net GND: track 458.2 -> 392.5 mm
- net A4: track 18.6 -> 58.5 mm
- net MS1: track 38.5 -> 0.00 mm
- net A2: track 9.42 -> 44.4 mm
- net MS2: track 34.5 -> 0.00 mm
- net A3: track 23.0 -> 54.9 mm
- net MS3: track 30.6 -> 0.00 mm
- net A1: track 9.42 -> 39.4 mm
- net A0: track 9.42 -> 35.4 mm
- net 12V: track 135.8 -> 160.9 mm
- net 5VOLTS: track 188.2 -> 206.9 mm
- net A6: track 0.00 -> 10.5 mm
- net A7: track 0.00 -> 10.5 mm
- net A5: track 0.00 -> 10.5 mm
- net 3V3: track 9.42 -> 0.00 mm
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Other:
- board size 88.9 x 87.6 mm -> 91.4 x 88.9 mm
