File: PCB/omnibot_board/v1/board_v1.sch (EAGLE design)
At the start: 15 parts, among them J1 292303-1

Commit message: changed v1 board
Parts:
- removed J5: (no value), SparkFun-Connectors:CONN_06SILK_FEMALE_PTH
- added J11: (no value), SparkFun-Connectors:CONN_05
- J4, J6, J7: SPICEPREFIX E -> (none)
Connections:
- removed net MS1: DRIVER.MS1, NANO.A7
- removed net MS2: DRIVER.MS2, NANO.A6
- removed net MS3: DRIVER.MS3, NANO.A5
- new net A5: J11.3, NANO.A5
- new net A6: J11.4, NANO.A6
- new net A7: J11.5, NANO.A7
- net 3V3: no longer J5.3
- net 5VOLTS: now also J11.2; no longer J5.2
- net A0: now also DRIVER.MS3; no longer J5.4
- net A1: now also DRIVER.MS2; no longer J5.5
- net A2: now also DRIVER.MS1; no longer J5.6
- net GND: now also J11.1; no longer J5.1
Other:
- note removed: "Camera control Arduino Nano"
- note removed: "GPIO Digial and analog"
- note removed: "I2C connectors"
- note removed: "LMI"
- note removed: "Motor driver"
- note removed: "OMNI BOARD"
- note removed: "Power supply"
- moved on the sheet: 12VSOURCE, 5VSOURCE, DRIVER, J1, J10, J2, J3, J4, J6, J7, J8, J9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
